Commit message: Add robot tests and refactoring of robot

File: rviz_rendering_tests/ogre_media_resources/test_meshes/test.urdf (robot description, URDF)
Before this commit: robot test_robot, 1 links, 0 joints
Links:
- added link test_robot_link_head; visual sphere radius=1
- added link test_robot_link_left_arm; visual box size=1 3 1
- added link test_robot_link_right_arm; visual box size=1 3 1
- link test_robot_link: geometry collision box size=1 1 1; visual mesh filename=package://rviz_rendering_tests/test_meshes/pr2-base.dae
Joints:
- added joint test_robot_continuous: type continuous, parent test_robot_link, child test_robot_link_head, origin xyz=0 0 0 rpy=0 0 0, axis 0 0 1
- added joint test_robot_fixed1: type fixed, parent test_robot_link, child test_robot_link_right_arm, origin xyz=0 0 0 rpy=0 0 0
- added joint test_robot_fixed2: type fixed, parent test_robot_link, child test_robot_link_left_arm, origin xyz=0 0 0 rpy=0 0 0
